Commit message: Descartes planner implemented with collision detection taking into account waypoint tolerances and multiple TCPs. Initial results generated. Collision bug fixed-wolrd manager works now. Changes made to the tolwaypoint module. repeated waypoints at 360 do not appear

File: src/robot_utilities/urdf/ur_10e/ur10e.urdf (robot description, URDF)
Before this commit: robot ur10e, 10 links, 9 joints
Joints:
- joint world_joint: origin xyz=0.0 0.0 0.0 rpy=0.0 0.0 0.0 -> xyz=0.0 0.0 0.0 rpy=0.0 0.0 0

Commit message: Minor bug fixes

File: src/robot_utilities/urdf/ur_10e/ur10e.urdf (robot description, URDF)
Before this commit: robot ur10e, 10 links, 9 joints
Joints:
- joint world_joint: origin xyz=0.0 0.0 0.0 rpy=0.0 0.0 0 -> xyz=0.0 0.0 0.0 rpy=0.0 0.0 3.141592
