Commit message: path consistency newer version computes workspace distances as a weighted sum of position and orientation from qs to all end configurations and picks the minimum. If the path is out of singularity and fully reachable. This approach works for 100000 random paths in workspace.

File: src/pct/data/tools/ati.xacro (robot description, xacro)
@@ -1,8 +1,8 @@
 <?xml version="1.0"?>
 <robot name="ati">
-  <link name="ati_origin">
+  <link name="tool_origin">
     <visual>
       	<geometry>
-          	<mesh filename="package://beg_tut/meshes/ati_sphere_orig.stl"
+          	<mesh filename="package://pct/data/meshes/ati.stl"
                 scale="1 1 1"/>
       	</geometry>
